File: schematics/bp4.1.kicad_pcb (KiCad board)
At the start: 2 copper layers, 90 x 32.6 mm, 39 parts, among them J1 Left Pin Strip, J2 Right Pin Strip, J3 I/O Pin Strip, J4 Power Pins A, J5 Power Pins B, J6 Power Pins C, SW1 Power Switch, U1 TPS61220DCK, U2 LM321

Commit message: add "(voltage setter)" label to R2 in bp4.1
Other:
- board text added: "(voltage setter)"
Changed lines of the file:
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@@
   (general
     (thickness 1.6)
-    (drawings 92)
+    (drawings 93)
     (tracks 306)
     (zones 0)
@@
     )
   )
+  (gr_text "(voltage setter)" (at 100.711 38.4175) (layer F.SilkS)
+    (effects (font (size 0.5 0.5) (thickness 0.1)))
+  )
   (gr_text "D3 GND D2" (at 59.309 28.7655) (layer F.SilkS)
