File: schematics/bp3.2.kicad_pcb (KiCad board)
At the start: 2 copper layers, 69.5 x 25 mm, 56 parts, among them J1 PowerInput, J2 PowerPassThru, J3 OutputPins, U1 INA128, U2 INA128, U3 INA128, U4 INA128

Commit message: minor tweaks to bp3.2
Other:
- board text added: "rectangles around R9-R12 indicate gain resistors"
- board text removed: "rectangles indicate gain resistors"
Changed lines of the file:
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@@
   (general
     (thickness 1.6)
-    (drawings 108)
+    (drawings 104)
     (tracks 402)
     (zones 0)
@@
     (effects (font (size 1 1) (thickness 0.15)) (justify left))
   )
-  (gr_line (start 82.4865 35.7505) (end 25.019 41.2115) (layer Cmts.User) (width 0.15))
-  (gr_line (start 72.9615 40.767) (end 25.146 41.5925) (layer Cmts.User) (width 0.15))
-  (gr_line (start 42.545 36.2585) (end 24.0665 40.513) (layer Cmts.User) (width 0.15))
-  (gr_line (start 32.8295 39.8145) (end 23.8125 41.021) (layer Cmts.User) (width 0.15))
-  (gr_text "rectangles\nindicate gain\nresistors" (at 17.8435 42.164) (layer Cmts.User)
+  (gr_text "rectangles around R9-R12\nindicate gain resistors" (at 37.2745 20.7645) (layer Cmts.User)
     (effects (font (size 1 1) (thickness 0.15)))
   )
