File: schematics/b4/PsyLinkMCP.kicad_pcb (KiCad board)
At the start: 2 copper layers, 70 x 25 mm, 65 parts, among them J1 PowerInput, J2 PowerPassThru, J3 OutputPins, U10 MCP6N11, U20 MCP6N11, U30 MCP6N11, U40 MCP6N11

Commit message: change labels (b3.2->b4, c10.2->c13)
Other:
- net class Default removed
- net class Power removed
- board text added: "psylink.me/b4"
- board text removed: "psylink.me/b3.2"
