File: schematics/electrode_module3.3/electrode_module3.3.kicad_sch (KiCad schematic)
At the start: 55 parts, among them J1 PowerInput, J2 PowerPassThru, J3 OutputPins, U1 INA128, U2 INA128, U3 INA128, U4 INA128

Commit message: fix gain resistor in circuit c10.3 (now c10.4)
Parts:
- R11, R12, R9: value 100/1% -> 200/1%
Other:
- note added: "Differential Amplifiers x4 Gain: 251x (Formula: 1+(50kOhm / RG) where RG = R9/10/11/12 = 200 Ohm)"
- note added: "https://psylink.me/c10.4"
- note removed: "Differential Amplifiers x4"
- note removed: "Note: R10 has 200 Ohms, lowering gain by half, compensating an interference bug on the out2 trace of PCBs B3.X"
- note removed: "https://psylink.me/c10.3"
- moved on the sheet: C1, C10, C2, C3, C4, C9, R1, R10, R2, R3, R4, R9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
